File: projects/RGB-TestPatternGenerator/RGB-TestPatternGenerator.brd (EAGLE design)
At the start: 100 x 80 mm, 48 parts, among them IC1 7805TV, IC2 7809TV, IC3 4060N, IC4 4040N, IC5 74HC10N, IC6 4082N, IC7 74HC32N, IC8 74LS157N, X1 D-SUB15-HDR15RA, Y1 8MHz

Commit message: feat: rgb layout
chnages:
- schematic modified
- layout modified
Connections:
- removed net VDD: IC3.16, IC4.16, IC6.14
- removed net VSS: IC3.8, IC4.8, IC6.7
- new net +5V: C3.+, C5.1, IC1.3, IC3.16, IC4.16, IC5.10, IC5.14, IC6.14, IC7.14, IC8.16, R14.2, R15.2, R16.2
- net GND: now also IC3.8, IC4.8, IC6.7, U$1.8
- net VCC: no longer C3.+, C5.1, IC1.3, IC5.10, IC5.14, IC7.14, IC8.16, R14.2, R15.2, R16.2
Changed lines of the file:
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@@
 </elements>
 <signals>
-<signal name="VSS">
-<contactref element="IC3" pad="8"/>
-<contactref element="IC4" pad="8"/>
-<contactref element="IC6" pad="7"/>
-<wire x1="-15.24" y1="27.94" x2="-57.15" y2="2.54" width="0" layer="19" extent="1-1"/>
-<wire x1="-15.24" y1="39.37" x2="-15.24" y2="27.94" width="0" layer="19" extent="1-1"/>
-</signal>
-<signal name="VDD">
-<contactref element="IC3" pad="16"/>
-<contactref element="IC4" pad="16"/>
-<contactref element="IC6" pad="14"/>
-<wire x1="-33.02" y1="35.56" x2="-74.93" y2="10.16" width="0" layer="19" extent="1-1"/>
-<wire x1="-30.48" y1="46.99" x2="-33.02" y2="35.56" width="0" layer="19" extent="1-1"/>
+<signal name="N$1">
+<contactref element="PWR" pad="MP"/>
+<contactref element="C1" pad="+"/>
+<contactref element="IC2" pad="1"/>
+<wire x1="-45.72" y1="54.61" x2="-29.21" y2="91.44" width="0" layer="19" extent="1-1"/>
+<wire x1="-64.77" y1="43.18" x2="-45.72" y2="54.61" width="0" layer="19" extent="1-1"/>
 </signal>
 <signal name="GND">
-<contactref element="IC5" pad="7"/>
-<contactref element="IC7" pad="7"/>
-<contactref element="IC8" pad="8"/>
 <contactref element="GND" pad="MP"/>
 <contactref element="C1" pad="-"/>
@@
 <contactref element="X1" pad="5"/>
 <contactref element="U$1" pad="2"/>
+<contactref element="U$1" pad="8"/>
+<contactref element="IC3" pad="8"/>
+<contactref element="IC4" pad="8"/>
+<contactref element="IC5" pad="7"/>
+<contactref element="IC6" pad="7"/>
+<contactref element="IC7" pad="7"/>
+<contactref element="IC8" pad="8"/>
 <wire x1="-36.83" y1="81.28" x2="-34.29" y2="91.44" width="0" layer="19" extent="1-1"/>
 <wire x1="-31.75" y1="71.12" x2="-36.83" y2="81.28" width="0" layer="19" extent="1-1"/>
@@
 <wire x1="-43.18" y1="54.61" x2="-31.75" y2="54.61" width="0" layer="19" extent="1-1"/>
 <wire x1="-17.78" y1="54.61" x2="-31.75" y2="54.61" width="0" layer="19" extent="1-1"/>
-<wire x1="-35.56" y1="39.37" x2="-31.75" y2="54.61" width="0" layer="19" extent="1-1"/>
-<wire x1="-38.1" y1="27.94" x2="-35.56" y2="39.37" width="0" layer="19" extent="1-1"/>
-<wire x1="-44.196" y1="20.32" x2="-38.1" y2="27.94" width="0" layer="19" extent="1-1"/>
-<wire x1="-43.053" y1="17.78" x2="-44.196" y2="20.32" width="0" layer="19" extent="1-1"/>
-<wire x1="-38.481" y1="17.78" x2="-43.053" y2="17.78" width="0" layer="19" extent="1-1"/>
-<wire x1="-36.195" y1="17.78" x2="-38.481" y2="17.78" width="0" layer="19" extent="1-1"/>
-<wire x1="-33.909" y1="17.78" x2="-36.195" y2="17.78" width="0" layer="19" extent="1-1"/>
-<wire x1="-22.03" y1="19.05" x2="-33.909" y2="17.78" width="0" layer="19" extent="1-1"/>
-<wire x1="-20.32" y1="35.56" x2="-35.56" y2="39.37" width="0" layer="19" extent="1-1"/>
+<wire x1="-15.24" y1="39.37" x2="-17.78" y2="54.61" width="0" layer="19" extent="1-1"/>
+<wire x1="-20.32" y1="35.56" x2="-15.24" y2="39.37" width="0" layer="19" extent="1-1"/>
+<wire x1="-15.24" y1="27.94" x2="-20.32" y2="35.56" width="0" layer="19" extent="1-1"/>
+<wire x1="-22.03" y1="19.05" x2="-15.24" y2="27.94" width="0" layer="19" extent="1-1"/>
+<wire x1="-33.909" y1="17.78" x2="-22.03" y2="19.05" width="0" layer="19" extent="1-1"/>
+<wire x1="-36.195" y1="17.78" x2="-33.909" y2="17.78" width="0" layer="19" extent="1-1"/>
+<wire x1="-38.481" y1="17.78" x2="-36.195" y2="17.78" width="0" layer="19" extent="1-1"/>
+<wire x1="-43.053" y1="17.78" x2="-38.481" y2="17.78" width="0" layer="19" extent="1-1"/>
+<wire x1="-44.196" y1="20.32" x2="-43.053" y2="17.78" width="0" layer="19" extent="1-1"/>
+<wire x1="-38.1" y1="27.94" x2="-44.196" y2="20.32" width="0" layer="19" extent="1-1"/>
+<wire x1="-35.56" y1="39.37" x2="-38.1" y2="27.94" width="0" layer="19" extent="1-1"/>
+<wire x1="-22.03" y1="3.81" x2="-22.03" y2="19.05" width="0" layer="19" extent="1-1"/>
 <wire x1="-60.96" y1="27.94" x2="-44.196" y2="20.32" width="0" layer="19" extent="1-1"/>
 <wire x1="-59.69" y1="43.18" x2="-60.96" y2="27.94" width="0" layer="19" extent="1-1"/>
@@
 <wire x1="-74.93" y1="76.2" x2="-67.31" y2="63.5" width="0" layer="19" extent="1-1"/>
 <wire x1="-64.77" y1="10.16" x2="-60.96" y2="27.94" width="0" layer="19" extent="1-1"/>
+<wire x1="-57.15" y1="2.54" x2="-64.77" y2="10.16" width="0" layer="19" extent="1-1"/>
 </signal>
 <signal name="VCC">
-<contactref element="IC5" pad="14"/>
-<contactref element="IC7" pad="14"/>
-<contactref element="IC8" pad="16"/>
 <contactref element="IC2" pad="3"/>
 <contactref element="C2" pad="+"/>
 <contactref element="C4" pad="1"/>
 <contactref element="IC1" pad="1"/>
-<contactref element="IC1" pad="3"/>
-<contactref element="C3" pad="+"/>
-<contactref element="C5" pad="1"/>
-<contactref element="R16" pad="2"/>
-<contactref element="R15" pad="2"/>
-<contactref element="R14" pad="2"/>
-<contactref element="IC5" pad="10"/>
 <contactref element="U$1" pad="14"/>
-<wire x1="-26.67" y1="86.36" x2="-13.97" y2="86.36" width="0" layer="19" extent="1-1"/>
-<wire x1="-39.37" y1="86.36" x2="-26.67" y2="86.36" width="0" layer="19" extent="1-1"/>
-<wire x1="-40.64" y1="54.61" x2="-39.37" y2="86.36" width="0" layer="19" extent="1-1"/>
+<wire x1="-74.93" y1="52.07" x2="-77.47" y2="43.18" width="0" layer="19" extent="1-1"/>
+<wire x1="-40.64" y1="54.61" x2="-74.93" y2="52.07" width="0" layer="19" extent="1-1"/>
 <wire x1="-34.29" y1="54.61" x2="-40.64" y2="54.61" width="0" layer="19" extent="1-1"/>
-<wire x1="-29.21" y1="54.61" x2="-34.29" y2="54.61" width="0" layer="19" extent="1-1"/>
-<wire x1="-22.86" y1="54.61" x2="-29.21" y2="54.61" width="0" layer="19" extent="1-1"/>
-<wire x1="-50.8" y1="46.99" x2="-40.64" y2="54.61" width="0" layer="19" extent="1-1"/>
-<wire x1="-55.88" y1="35.56" x2="-50.8" y2="46.99" width="0" layer="19" extent="1-1"/>
-<wire x1="-66.04" y1="35.56" x2="-55.88" y2="35.56" width="0" layer="19" extent="1-1"/>
-<wire x1="-76.2" y1="35.56" x2="-66.04" y2="35.56" width="0" layer="19" extent="1-1"/>
-<wire x1="-77.47" y1="43.18" x2="-76.2" y2="35.56" width="0" layer="19" extent="1-1"/>
-<wire x1="-74.93" y1="52.07" x2="-77.47" y2="43.18" width="0" layer="19" extent="1-1"/>
-<wire x1="-82.55" y1="52.07" x2="-74.93" y2="52.07" width="0" layer="19" extent="1-1"/>
-<wire x1="-13.53" y1="16.51" x2="-22.86" y2="54.61" width="0" layer="19" extent="1-1"/>
-</signal>
-<signal name="N$1">
-<contactref element="PWR" pad="MP"/>
-<contactref element="C1" pad="+"/>
-<contactref element="IC2" pad="1"/>
-<wire x1="-45.72" y1="54.61" x2="-29.21" y2="91.44" width="0" layer="19" extent="1-1"/>
-<wire x1="-64.77" y1="43.18" x2="-45.72" y2="54.61" width="0" layer="19" extent="1-1"/>
+<wire x1="-13.53" y1="16.51" x2="-34.29" y2="54.61" width="0" layer="19" extent="1-1"/>
 </signal>
 <signal name="N$2">
@@
 <wire x1="-13.53" y1="6.35" x2="-13.53" y2="11.43" width="0" layer="19" extent="1-1"/>
 </signal>
+<signal name="+5V">
+<contactref element="IC1" pad="3"/>
+<contactref element="C3" pad="+"/>
+<contactref element="C5" pad="1"/>
+<contactref element="R16" pad="2"/>
+<contactref element="R15" pad="2"/>
+<contactref element="R14" pad="2"/>
+<contactref element="IC5" pad="10"/>
+<contactref element="IC3" pad="16"/>
+<contactref element="IC4" pad="16"/>
+<contactref element="IC5" pad="14"/>
+<contactref element="IC6" pad="14"/>
+<contactref element="IC7" pad="14"/>
+<contactref element="IC8" pad="16"/>
+<wire x1="-26.67" y1="86.36" x2="-13.97" y2="86.36" width="0" layer="19" extent="1-1"/>
+<wire x1="-39.37" y1="86.36" x2="-26.67" y2="86.36" width="0" layer="19" extent="1-1"/>
+<wire x1="-29.21" y1="54.61" x2="-26.67" y2="86.36" width="0" layer="19" extent="1-1"/>
+<wire x1="-22.86" y1="54.61" x2="-29.21" y2="54.61" width="0" layer="19" extent="1-1"/>
+<wire x1="-30.48" y1="46.99" x2="-29.21" y2="54.61" width="0" layer="19" extent="1-1"/>
+<wire x1="-33.02" y1="35.56" x2="-30.48" y2="46.99" width="0" layer="19" extent="1-1"/>
+<wire x1="-50.8" y1="46.99" x2="-30.48" y2="46.99" width="0" layer="19" extent="1-1"/>
+<wire x1="-55.88" y1="35.56" x2="-50.8" y2="46.99" width="0" layer="19" extent="1-1"/>
+<wire x1="-66.04" y1="35.56" x2="-55.88" y2="35.56" width="0" layer="19" extent="1-1"/>
+<wire x1="-76.2" y1="35.56" x2="-66.04" y2="35.56" width="0" layer="19" extent="1-1"/>
+<wire x1="-82.55" y1="52.07" x2="-76.2" y2="35.56" width="0" layer="19" extent="1-1"/>
+<wire x1="-74.93" y1="10.16" x2="-76.2" y2="35.56" width="0" layer="19" extent="1-1"/>
+</signal>
 </signals>

Commit message: feat: rgb layout
Parts:
- moved C2 168.1 mm to (92.7, 55.9)
- moved C5 157.6 mm to (77.5, 57.1), turned to 90 degrees
- moved C4 156.3 mm to (83.8, 57.1), turned to 90 degrees
- moved R13 148.8 mm to (62.2, 12.7)
- moved R18 147.7 mm to (63.5, 22.9)
- moved C1 145.5 mm to (81.3, 67.3)
- moved R17 134.0 mm to (63.5, 27.9)
- moved IC2 126.3 mm to (81.3, 78.7)
- moved IC1 126.3 mm to (92.7, 78.7)
- moved X1 124.8 mm to (85.1, 8.89)
- moved R12 121.6 mm to (50.8, 25.4)
- moved C3 113.7 mm to (92.7, 67.3)
- moved C7 111.9 mm to (41.9, 58.4), turned to 90 degrees
- moved C6 110.6 mm to (48.3, 58.4), turned to 90 degrees
- moved GND 107.8 mm to (72.4, 76.2)
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
Commit message: feat: rgb layout
Parts:
- moved R13 74.6 mm to (7.62, 63.5)
- moved R18 72.2 mm to (7.62, 68.6)
- moved R17 59.3 mm to (20.3, 68.6)
- moved R9 51.2 mm to (58.4, 63.5)
- moved R12 48.8 mm to (20.3, 63.5)
- moved R19 45.1 mm to (58.4, 73.7)
- moved C10 40.7 mm to (45.7, 45.7)
- moved C8 40.7 mm to (61.0, 45.7)
- moved C9 40.7 mm to (53.3, 45.7)
- moved R14 37.6 mm to (58.4, 68.6)
- moved C7 36.6 mm to (7.62, 45.7), turned to 0 degrees
- moved C6 35.4 mm to (15.2, 45.7), turned to 0 degrees
- moved R10 26.2 mm to (45.7, 63.5)
- moved C11 19.9 mm to (38.1, 45.7)
- moved C12 19.9 mm to (30.5, 45.7)
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Routing:
- net GND: track 0.00 -> 410.7 mm
- net +5V: track 0.00 -> 222.3 mm, vias 0 -> 1
- net N$38: track 0.00 -> 129.0 mm
- net N$34: track 0.00 -> 117.8 mm, vias 0 -> 1
- net N$36: track 0.00 -> 108.2 mm
- net N$41: track 0.00 -> 107.9 mm, vias 0 -> 1
- net N$3: track 0.00 -> 107.8 mm
- net N$35: track 0.00 -> 95.4 mm, vias 0 -> 1
- net N$32: track 0.00 -> 95.2 mm
- net N$37: track 0.00 -> 93.0 mm, vias 0 -> 1
- net N$2: track 0.00 -> 88.1 mm
- net N$33: track 0.00 -> 85.9 mm
- net VCC: track 0.00 -> 84.3 mm
- net N$40: track 0.00 -> 74.6 mm, vias 0 -> 1
- net N$4: track 0.00 -> 73.9 mm, vias 0 -> 2
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
Commit message: well well well
Parts:
- moved R18 93.7 mm to (86.4, 17.8), turned to 45 degrees
- moved R17 88.4 mm to (92.7, 17.8), turned to 45 degrees
- moved C4 80.4 mm to (3.81, 64.8)
- moved C2 72.1 mm to (22.9, 73.7)
- moved R13 71.9 mm to (61.0, 15.2), turned to 45 degrees
- moved C1 70.1 mm to (11.4, 73.7)
- moved GND 69.8 mm to (2.54, 76.2)
- moved C5 67.7 mm to (10.2, 64.8)
- moved R12 67.1 mm to (61.0, 10.2), turned to 45 degrees
- moved PWR 65.0 mm to (2.54, 71.1)
- moved R8 63.5 mm to (69.8, 45.7), turned to 45 degrees
- moved R19 59.9 mm to (80.0, 17.8), turned to 45 degrees
- moved C3 58.8 mm to (34.3, 73.7)
- moved R7 55.7 mm to (61.0, 20.3), turned to 45 degrees
- moved C13 54.6 mm to (77.5, 44.5), turned to 45 degrees
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Routing:
- net GND: track 410.7 -> 0.00 mm
- net +5V: track 222.3 -> 0.00 mm, vias 1 -> 0
- net N$38: track 129.0 -> 0.00 mm
- net N$34: track 117.8 -> 0.00 mm, vias 1 -> 0
- net N$36: track 108.2 -> 0.00 mm
- net N$41: track 107.9 -> 0.00 mm, vias 1 -> 0
- net N$3: track 107.8 -> 0.00 mm
- net N$35: track 95.4 -> 0.00 mm, vias 1 -> 0
- net N$32: track 95.2 -> 0.00 mm
- net N$37: track 93.0 -> 0.00 mm, vias 1 -> 0
- net N$2: track 88.1 -> 0.00 mm
- net N$33: track 85.9 -> 0.00 mm
- net VCC: track 84.3 -> 0.00 mm
- net N$40: track 74.6 -> 0.00 mm, vias 1 -> 0
- net N$4: track 73.9 -> 0.00 mm, vias 2 -> 0
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
Commit message: well, this should do it for now ..
Routing:
- net GND: track 0.00 -> 367.5 mm
- net +5V: track 0.00 -> 206.9 mm
- net VCC: track 0.00 -> 122.8 mm
- net N$37: track 0.00 -> 110.7 mm
- net N$8: track 0.00 -> 86.3 mm
- net N$12: track 0.00 -> 81.3 mm
- net N$10: track 0.00 -> 77.3 mm
- net N$32: track 0.00 -> 75.1 mm
- net N$9: track 0.00 -> 66.9 mm
- net N$1: track 0.00 -> 65.2 mm
- net N$4: track 0.00 -> 59.0 mm
- net N$11: track 0.00 -> 58.9 mm
- net N$18: track 0.00 -> 56.2 mm
- net N$33: track 0.00 -> 53.8 mm
- net N$28: track 0.00 -> 52.6 mm
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