File: projects/PowerSupply/PLCPart.brd (EAGLE design)
At the start: 100 x 80 mm, 44 parts, among them IC1 L7818CV, IC2 L7918CV, IC3 LM2574N-5.0, IC4 LM2574N-5.0, IC5 L7915CV, IC6 L7815CV, IC7 LM358N, IC8 LM358N, X1 MCU-PWR, X2 MCU-IN, X4 MCU-OUT

Commit message: feat: plc part modified
Parts:
- C14, C16: value 220µF -> 470µF
- L1, L2: value 33µH -> 68µH; device inductor-neosid:SD12-680 -> inductor-neosid:SD12K100
- moved L2 64.4 mm to (-2.50, -51.0)
- moved L1 47.7 mm to (-2.50, -38.3)
Changed lines of the file:
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@@
 <attribute name="VALUE" x="-63.5" y="52.451" size="1.27" layer="27" ratio="10"/>
 </element>
-<element name="C14" library="rcl" library_urn="urn:adsk.eagle:library:334" package="E2-5" package3d_urn="urn:adsk.eagle:package:23346/2" value="220µF" x="-44.45" y="54.61" smashed="yes">
+<element name="C14" library="rcl" library_urn="urn:adsk.eagle:library:334" package="E2-5" package3d_urn="urn:adsk.eagle:package:23346/2" value="470µF" x="-44.45" y="54.61" smashed="yes">
 <attribute name="NAME" x="-41.91" y="55.626" size="1.27" layer="25" ratio="10"/>
 <attribute name="POPULARITY" value="14" x="0" y="0" size="1.778" layer="27" display="off"/>
@@
 <attribute name="VALUE" x="-17.78" y="60.071" size="1.27" layer="27" ratio="10"/>
 </element>
-<element name="C16" library="rcl" library_urn="urn:adsk.eagle:library:334" package="E2-5" package3d_urn="urn:adsk.eagle:package:23346/2" value="220µF" x="-55.88" y="54.61" smashed="yes">
+<element name="C16" library="rcl" library_urn="urn:adsk.eagle:library:334" package="E2-5" package3d_urn="urn:adsk.eagle:package:23346/2" value="470µF" x="-55.88" y="54.61" smashed="yes">
 <attribute name="NAME" x="-53.34" y="55.626" size="1.27" layer="25" ratio="10"/>
 <attribute name="POPULARITY" value="14" x="0" y="0" size="1.778" layer="27" display="off"/>
@@
 <attribute name="VALUE" x="-73.66" y="26.67" size="1.27" layer="27" ratio="10"/>
 </element>
-<element name="L1" library="inductor-neosid" library_urn="urn:adsk.eagle:library:241" package="SD12-680" package3d_urn="urn:adsk.eagle:package:14657/1" value="33µH" x="-19.05" y="6.35" smashed="yes">
-<attribute name="MF" value="BUSSMANN" x="0" y="0" size="1.778" layer="27" display="off"/>
-<attribute name="MPN" value="SD12-680" x="0" y="0" size="1.778" layer="27" display="off"/>
-<attribute name="NAME" x="-15.323" y="11.398" size="1.27" layer="25"/>
-<attribute name="OC_FARNELL" value="unknown" x="0" y="0" size="1.778" layer="27" display="off"/>
-<attribute name="OC_NEWARK" value="19K7201" x="0" y="0" size="1.778" layer="27" display="off"/>
-<attribute name="POPULARITY" value="0" x="0" y="0" size="1.778" layer="27" display="off"/>
-<attribute name="VALUE" x="-22.3" y="3.35" size="1.27" layer="27"/>
-</element>
-<element name="L2" library="inductor-neosid" library_urn="urn:adsk.eagle:library:241" package="SD12-680" package3d_urn="urn:adsk.eagle:package:14657/1" value="33µH" x="-31.75" y="6.35" smashed="yes">
-<attribute name="MF" value="BUSSMANN" x="0" y="0" size="1.778" layer="27" display="off"/>
-<attribute name="MPN" value="SD12-680" x="0" y="0" size="1.778" layer="27" display="off"/>
-<attribute name="NAME" x="-28.023" y="11.398" size="1.27" layer="25"/>
-<attribute name="OC_FARNELL" value="unknown" x="0" y="0" size="1.778" layer="27" display="off"/>
-<attribute name="OC_NEWARK" value="19K7201" x="0" y="0" size="1.778" layer="27" display="off"/>
-<attribute name="POPULARITY" value="0" x="0" y="0" size="1.778" layer="27" display="off"/>
-<attribute name="VALUE" x="-35" y="3.35" size="1.27" layer="27"/>
+<element name="L1" library="inductor-neosid" library_urn="urn:adsk.eagle:library:241" package="SD12K100" package3d_urn="urn:adsk.eagle:package:14651/1" value="68µH" x="-2.5" y="-38.335" smashed="yes">
+<attribute name="MF" value="" x="16.55" y="-44.685" size="1.778" layer="27" display="off"/>
+<attribute name="MPN" value="" x="16.55" y="-44.685" size="1.778" layer="27" display="off"/>
+<attribute name="NAME" x="1.227" y="-33.287" size="1.27" layer="25"/>
+<attribute name="OC_FARNELL" value="unknown" x="16.55" y="-44.685" size="1.778" layer="27" display="off"/>
+<attribute name="OC_NEWARK" value="unknown" x="16.55" y="-44.685" size="1.778" layer="27" display="off"/>
+<attribute name="POPULARITY" value="0" x="16.55" y="-44.685" size="1.778" layer="27" display="off"/>
+<attribute name="VALUE" x="-5.75" y="-41.335" size="1.27" layer="27"/>
+</element>
+<element name="L2" library="inductor-neosid" library_urn="urn:adsk.eagle:library:241" package="SD12K100" package3d_urn="urn:adsk.eagle:package:14651/1" value="68µH" x="-2.5" y="-51.035" smashed="yes">
+<attribute name="MF" value="" x="29.25" y="-57.385" size="1.778" layer="27" display="off"/>
+<attribute name="MPN" value="" x="29.25" y="-57.385" size="1.778" layer="27" display="off"/>
+<attribute name="NAME" x="1.227" y="-45.987" size="1.27" layer="25"/>
+<attribute name="OC_FARNELL" value="unknown" x="29.25" y="-57.385" size="1.778" layer="27" display="off"/>
+<attribute name="OC_NEWARK" value="unknown" x="29.25" y="-57.385" size="1.778" layer="27" display="off"/>
+<attribute name="POPULARITY" value="0" x="29.25" y="-57.385" size="1.778" layer="27" display="off"/>
+<attribute name="VALUE" x="-5.75" y="-54.035" size="1.27" layer="27"/>
 </element>
 <element name="R1" library="rcl" library_urn="urn:adsk.eagle:library:334" package="0207/10" package3d_urn="urn:adsk.eagle:package:23491/2" value="10k" x="-29.21" y="60.96" smashed="yes">
@@
 <wire x1="-52.07" y1="67.31" x2="-56.896" y2="54.61" width="0" layer="19" extent="1-1"/>
 <wire x1="-25.4" y1="27.94" x2="-45.466" y2="54.61" width="0" layer="19" extent="1-1"/>
-<wire x1="-26.75" y1="6.35" x2="-25.4" y2="27.94" width="0" layer="19" extent="1-1"/>
-<wire x1="-14.05" y1="6.35" x2="-26.75" y2="6.35" width="0" layer="19" extent="1-1"/>
-<wire x1="-63.5" y1="15.24" x2="-26.75" y2="6.35" width="0" layer="19" extent="1-1"/>
+<wire x1="-63.5" y1="15.24" x2="-56.896" y2="54.61" width="0" layer="19" extent="1-1"/>
+<wire x1="0" y1="-38.335" x2="-25.4" y2="27.94" width="0" layer="19" extent="1-1"/>
+<wire x1="0" y1="-51.035" x2="0" y2="-38.335" width="0" layer="19" extent="1-1"/>
 </signal>
 <signal name="N$2">
@@
 <contactref element="IC3" pad="7"/>
 <contactref element="L1" pad="1"/>
-<wire x1="-24.05" y1="6.35" x2="-60.96" y2="22.86" width="0" layer="19" extent="1-1"/>
-<wire x1="-24.13" y1="40.64" x2="-24.05" y2="6.35" width="0" layer="19" extent="1-1"/>
+<wire x1="-24.13" y1="40.64" x2="-5" y2="-38.335" width="0" layer="19" extent="1-1"/>
+<wire x1="-60.96" y1="22.86" x2="-24.13" y2="40.64" width="0" layer="19" extent="1-1"/>
 </signal>
 <signal name="N$6">
@@
 <contactref element="IC4" pad="7"/>
 <contactref element="L2" pad="1"/>
-<wire x1="-22.86" y1="35.56" x2="-36.75" y2="6.35" width="0" layer="19" extent="1-1"/>
+<wire x1="-22.86" y1="35.56" x2="-5" y2="-51.035" width="0" layer="19" extent="1-1"/>
 <wire x1="-35.56" y1="40.64" x2="-22.86" y2="35.56" width="0" layer="19" extent="1-1"/>
 </signal>
